Commit message: Make box longer along z-axis, fix position of handle.

File: urdf/box.urdf (robot description, URDF)
Before this commit: robot box, 1 links, 0 joints
Links:
- link base_link: geometry collision box size=0.05 0.05 0.1; visual box size=0.05 0.05 0.1

Commit message: Add a box with colors and a cup

File: urdf/box.urdf (robot description, URDF)
Before this commit: robot box, 1 links, 0 joints
Links:
- link base_link: mass None -> 0.6; geometry collision box size=0.03 0.05 0.05; visual box size=0.03 0.05 0.05
