Commit message: Remove collision geometry for base_footprint.

File: urdf/pr2.urdf (robot description, URDF)
Before this commit: robot pr2, 82 links, 81 joints
Links:
- link base_footprint: geometry visual box size=0.01 0.01 0.01

Commit message: Remove collision geometry for some more fixed objects.

File: urdf/pr2.urdf (robot description, URDF)
Before this commit: robot pr2, 82 links, 81 joints
Links:
- link base_laser_link: geometry visual box size=0.001 0.001 0.001
- link head_plate_frame: geometry visual box size=0.01 0.01 0.01
- link high_def_frame: geometry visual box size=0.04 0.04 0.04
- link high_def_optical_frame: geometry visual cylinder length=0.05 radius=0.02
- link imu_link: geometry visual box size=0.001 0.001 0.001
- link l_forearm_cam_frame: geometry visual box size=0.01 0.01 0.01
- link l_gripper_motor_accelerometer_link: geometry visual box size=0.001 0.001 0.001
- link l_wrist_roll_link: geometry visual mesh filename=package://pr2_description/meshes/forearm_v0/wrist_roll.stl
- link laser_tilt_link: geometry visual box size=0.001 0.001 0.001
- link narrow_stereo_gazebo_l_stereo_camera_frame: geometry visual box size=0.01 0.01 0.01
- link narrow_stereo_gazebo_r_stereo_camera_frame: geometry visual box size=0.01 0.01 0.01
- link narrow_stereo_link: geometry visual box size=0.001 0.001 0.001
- link r_forearm_cam_frame: geometry visual box size=0.01 0.01 0.01
- link r_gripper_motor_accelerometer_link: geometry visual box size=0.001 0.001 0.001
- link r_wrist_roll_link: geometry visual mesh filename=package://pr2_description/meshes/forearm_v0/wrist_roll.stl
- link sensor_mount_link: geometry visual box size=0.01 0.01 0.01
- link wide_stereo_gazebo_l_stereo_camera_frame: geometry visual box size=0.01 0.01 0.01
- link wide_stereo_gazebo_r_stereo_camera_frame: geometry visual box size=0.01 0.01 0.01
- link wide_stereo_link: geometry visual box size=0.001 0.001 0.001

Commit message: Remove collision geometry for x_gripper_y_parallel_link.
  for x, y in {"l", "r"}.

File: urdf/pr2.urdf (robot description, URDF)
Before this commit: robot pr2, 82 links, 81 joints
Links:
- link l_gripper_l_parallel_link: geometry 
- link l_gripper_r_parallel_link: geometry 
- link r_gripper_l_parallel_link: geometry 
- link r_gripper_r_parallel_link: geometry 

Commit message: Remove degrees of freedom of the wheels.

File: urdf/pr2.urdf (robot description, URDF)
Before this commit: robot pr2, 82 links, 81 joints
Joints:
- joint bl_caster_l_wheel_joint: type continuous -> fixed
- joint bl_caster_r_wheel_joint: type continuous -> fixed
- joint bl_caster_rotation_joint: type continuous -> fixed
- joint br_caster_l_wheel_joint: type continuous -> fixed
- joint br_caster_r_wheel_joint: type continuous -> fixed
- joint br_caster_rotation_joint: type continuous -> fixed
- joint fl_caster_l_wheel_joint: type continuous -> fixed
- joint fl_caster_r_wheel_joint: type continuous -> fixed
- joint fl_caster_rotation_joint: type continuous -> fixed
- joint fr_caster_l_wheel_joint: type continuous -> fixed
- joint fr_caster_r_wheel_joint: type continuous -> fixed
- joint fr_caster_rotation_joint: type continuous -> fixed

Commit message: Remove collision geometry of the wheels.

File: urdf/pr2.urdf (robot description, URDF)
Before this commit: robot pr2, 82 links, 81 joints
Links:
- link bl_caster_l_wheel_link: geometry visual mesh filename=package://pr2_description/meshes/base_v0/wheel.stl
- link bl_caster_r_wheel_link: geometry visual mesh filename=package://pr2_description/meshes/base_v0/wheel.stl
- link bl_caster_rotation_link: geometry visual mesh filename=package://pr2_description/meshes/base_v0/caster.stl
- link br_caster_l_wheel_link: geometry visual mesh filename=package://pr2_description/meshes/base_v0/wheel.stl
- link br_caster_r_wheel_link: geometry visual mesh filename=package://pr2_description/meshes/base_v0/wheel.stl
- link br_caster_rotation_link: geometry visual mesh filename=package://pr2_description/meshes/base_v0/caster.stl
- link fl_caster_l_wheel_link: geometry visual mesh filename=package://pr2_description/meshes/base_v0/wheel.stl
- link fl_caster_r_wheel_link: geometry visual mesh filename=package://pr2_description/meshes/base_v0/wheel.stl
- link fl_caster_rotation_link: geometry visual mesh filename=package://pr2_description/meshes/base_v0/caster.stl
- link fr_caster_l_wheel_link: geometry visual mesh filename=package://pr2_description/meshes/base_v0/wheel.stl
- link fr_caster_r_wheel_link: geometry visual mesh filename=package://pr2_description/meshes/base_v0/wheel.stl
- link fr_caster_rotation_link: geometry visual mesh filename=package://pr2_description/meshes/base_v0/caster.stl

Commit message: Update to integration of pinocchio

File: urdf/pr2.urdf (robot description, URDF)
Before this commit: robot pr2, 82 links, 81 joints
Joints:
- joint l_gripper_joint: type prismatic -> fixed
- joint r_gripper_joint: type prismatic -> fixed
